File: AD9854_SDR/kicad_AD9854_demo1/AD9854_demo1.kicad_pcb (KiCad board)
At the start: 2 copper layers, 100.1 x 57.5 mm, 51 parts, among them U1 AD9854ASTZ, U2 LT5560, U3 MCP1826ST-3302E/EB, X1 OSC5A2B02, Y1 ECS-2520MV-xxx-xx

Commit message: more
Parts:
- removed TR1: TRANSF5, Transformer_THT:Transformer_Toroid_Horizontal_D9.0mm_Amidon-T30
- removed X1: OSC5A2B02, Oscillator:Oscillator_DIP-8
- added C40: C, Capacitor_SMD:C_0603_1608Metric_Pad1.08x0.95mm_HandSolder, F.Cu at (104.5, 74.0)
- added C41: C, Capacitor_SMD:C_0603_1608Metric_Pad1.08x0.95mm_HandSolder, F.Cu at (104.5, 76.6)
- added C42: C, Capacitor_SMD:C_0603_1608Metric_Pad1.08x0.95mm_HandSolder, F.Cu at (104.5, 79.1)
- added C43: C, Capacitor_SMD:C_0603_1608Metric_Pad1.08x0.95mm_HandSolder, F.Cu at (104.5, 81.6)
- added C45: C, Capacitor_SMD:C_0603_1608Metric_Pad1.08x0.95mm_HandSolder, F.Cu at (104.5, 84.1)
- added C46: C, Capacitor_SMD:C_0603_1608Metric_Pad1.08x0.95mm_HandSolder, F.Cu at (108.9, 69.0)
- added C47: C, Capacitor_SMD:C_0603_1608Metric_Pad1.08x0.95mm_HandSolder, F.Cu at (108.9, 71.5)
- added C48: C, Capacitor_SMD:C_0603_1608Metric_Pad1.08x0.95mm_HandSolder, F.Cu at (108.9, 74.0)
- added C49: C, Capacitor_SMD:C_0603_1608Metric_Pad1.08x0.95mm_HandSolder, F.Cu at (108.9, 76.6)
- added C50: C, Capacitor_SMD:C_0603_1608Metric_Pad1.08x0.95mm_HandSolder, F.Cu at (108.9, 79.1)
- added C51: C, Capacitor_SMD:C_0603_1608Metric_Pad1.08x0.95mm_HandSolder, F.Cu at (108.9, 81.6)
- added C52: C, Capacitor_SMD:C_0603_1608Metric_Pad1.08x0.95mm_HandSolder, F.Cu at (108.9, 84.1)
- added C53: 0.01uF, Capacitor_SMD:C_0603_1608Metric_Pad1.08x0.95mm_HandSolder, F.Cu at (154.7, 99.5)
- added J1: Conn_Coaxial_Small, Connector_Coaxial:SMA_Amphenol_132289_EdgeMount, F.Cu at (117.6, 56.2)
- added J2: Conn_02x08_Row_Letter_First, Connector_PinHeader_1.27mm:PinHeader_2x08_P1.27mm_Horizontal, F.Cu at (226.5, 110.2)
- added K1: G6H-2, Relay_SMD:Relay_DPDT_Omron_G6H-2F, F.Cu at (125.8, 75.1)
- added L1: L, Inductor_SMD:L_0805_2012Metric_Pad1.15x1.40mm_HandSolder, F.Cu at (100.0, 69.2)
- added L2: L, Inductor_SMD:L_0805_2012Metric_Pad1.15x1.40mm_HandSolder, F.Cu at (100.0, 72.2)
- added L3: L, Inductor_SMD:L_0805_2012Metric_Pad1.15x1.40mm_HandSolder, F.Cu at (100.0, 75.2)
- added L4: L, Inductor_SMD:L_0805_2012Metric_Pad1.15x1.40mm_HandSolder, F.Cu at (100.0, 78.1)
- added L5: L, Inductor_SMD:L_0805_2012Metric_Pad1.15x1.40mm_HandSolder, F.Cu at (100.0, 81.0)
- added L6: L, Inductor_SMD:L_0805_2012Metric_Pad1.15x1.40mm_HandSolder, F.Cu at (100.0, 84.0)
- added Q1: AO3401A, Package_TO_SOT_SMD:SOT-23W_Handsoldering, F.Cu at (157.2, 53.2)
- added Q2: AO3400A, Package_TO_SOT_SMD:SOT-23, F.Cu at (164.7, 53.5)
- added R5: 3900, Resistor_SMD:R_0805_2012Metric_Pad1.20x1.40mm_HandSolder, F.Cu at (154.9, 96.7)
- added SW1: RotaryEncoder_Switch_MP, Rotary_Encoder:RotaryEncoder_Alps_EC12E-Switch_Vertical_H20mm_CircularMountingHoles, F.Cu at (244.7, 106.3)
- added SW2: SW_NKK_GW12LJPCF, Button_Switch_THT:SW_NKK_GW12LJP, F.Cu at (230.7, 57.3)
- added TR2: TRANSF3, Transformer_THT:Transformer_Toroid_Horizontal_D9.0mm_Amidon-T30, F.Cu at (112.0, 97.8)
- C1, C2: value 0.1uF -> C
- R1: value 330 -> R
- R2: value 100 -> R
- R3, R4: value 10k -> R
- U3: footprint MCP1826ST:DDPAK3_MC_MCH -> Package_TO_SOT_SMD:TO-263-2_TabPin1
- Y1: value ECS-2520MV-xxx-xx -> Si570; footprint Oscillator:Oscillator_SMD_ECS_2520MV-xxx-xx-4Pin_2.5x2.0mm -> Oscillator:Oscillator_SMD_SI570_SI571_HandSoldering
- moved C1 49.0 mm to (104.5, 69.0)
- moved C2 49.0 mm to (104.5, 71.5)
- moved R2 43.9 mm to (113.2, 71.5)
- moved R3 43.9 mm to (113.2, 74.0)
- moved R4 43.9 mm to (113.2, 76.6)
- moved R1 40.8 mm to (113.2, 69.0)
- moved U2 29.7 mm to (129.3, 94.0)
- moved C3 19.8 mm to (152.6, 63.9)
- moved A1 15.4 mm to (187.1, 76.4)
- moved Y1 13.3 mm to (159.2, 71.6)
Connections:
- C1 pad 1: Net-(C1-Pad1) -> I_out_A
- C1 pad 2: diffclockA -> GND
- C2 pad 1: GND -> I_out_A
- C2 pad 2: diffclockB -> Net-(C2-Pad2)
- R1 pad 1: Net-(C1-Pad1) -> I_out_B
- R1 pad 2: 5v_clock -> GND
- R2 pad 1: Net-(C1-Pad1) -> Q_out_B
- R3 pad 1: 3v_ldo -> diffclockA
- R3 pad 2: diffclockA -> GND
- R4 pad 1: diffclockA -> diffclockB
- U1 pad 14: unconnected-(U1-A5-Pad14) -> addrbus5
- U1 pad 15: unconnected-(U1-A4-Pad15) -> addrbus4
- U1 pad 16: unconnected-(U1-A3-Pad16) -> addrbus3
- U1 pad 17: unconnected-(U1-A2/IORESET-Pad17) -> addrbus2
- U1 pad 18: unconnected-(U1-A1/SDO-Pad18) -> addrbus1
- U1 pad 19: unconnected-(U1-A0/SDIO-Pad19) -> addrbus0
- U1 pad 20: unconnected-(U1-I/OUDCLK-Pad20) -> ioclock_AD9854
- U1 pad 21: unconnected-(U1-WR*/SCLK-Pad21) -> writeready_AD9854
- U1 pad 22: unconnected-(U1-RD*/CS*-Pad22) -> readdata_AD9854
- U1 pad 48: unconnected-(U1-IOUT1-Pad48) -> Q_out_A
- U1 pad 49: unconnected-(U1-IOUT1*-Pad49) -> Q_out_B
- U1 pad 51: unconnected-(U1-IOUT2*-Pad51) -> I_out_B
- U1 pad 52: unconnected-(U1-IOUT2-Pad52) -> I_out_A
- U1 pad 55: unconnected-(U1-DACBP-Pad55) -> Net-(U1-DACBP)
- U1 pad 64: unconnected-(U1-DIFFCLKENABLE-Pad64) -> 3.3v_AVDD
- U1 pad 70: unconnected-(U1-S/P_SELECT-Pad70) -> 3.3v_AVDD
- U1 pad 71: unconnected-(U1-MASTERRESET-Pad71) -> RESET_AD9854
- Y1 pad 2: GND -> unconnected-(Y1-OE-Pad2)
- Y1 pad 3: diffclockA -> GND
- Y1 pad 4: 3v_ldo -> diffclockA
Other:
- board size 100.1 x 57.5 mm -> 109.6 x 65.8 mm
