File: AD9854_SDR/kicad_AD9854_demo1/AD9854_demo1.kicad_sch (KiCad schematic)
At the start: 51 parts, among them U1 AD9854ASTZ, U2 LT5560, U3 MCP1826ST-3302E/EB, X1 OSC5A2B02, Y1 ECS-2520MV-xxx-xx

Commit message: more
Parts:
- removed C3: 0.1uF, Capacitor_SMD:C_0603_1608Metric_Pad1.08x0.95mm_HandSolder, symbol Device:C
- removed X1: OSC5A2B02, Oscillator:Oscillator_DIP-8, symbol osc5a2b02:OSC5A2B02
- removed Y1: ECS-2520MV-xxx-xx, Oscillator:Oscillator_SMD_ECS_2520MV-xxx-xx-4Pin_2.5x2.0mm, symbol Oscillator:ECS-2520MV-xxx-xx
- added C40, C41, C42, C43, C45, C46, C47, C48, C49, C50, C51, C52: C, Capacitor_SMD:C_0603_1608Metric_Pad1.08x0.95mm_HandSolder, symbol Device:C
- added C53: 0.01uF, Capacitor_SMD:C_0603_1608Metric_Pad1.08x0.95mm_HandSolder, symbol Device:C
- added J1: Conn_Coaxial_Small, Connector_Coaxial:SMA_Amphenol_132289_EdgeMount, symbol Connector:Conn_Coaxial_Small
- added J2: Conn_02x08_Row_Letter_First, Connector_PinHeader_1.27mm:PinHeader_2x08_P1.27mm_Horizontal, symbol Connector_Generic:Conn_02x08_Row_Letter_First
- added K1: G6H-2, Relay_SMD:Relay_DPDT_Omron_G6H-2F, symbol Relay:G6H-2
- added L1, L2, L3, L4, L5, L6: L, Inductor_SMD:L_0805_2012Metric_Pad1.15x1.40mm_HandSolder, symbol Device:L
- added Q1: AO3401A, Package_TO_SOT_SMD:SOT-23W_Handsoldering, symbol Transistor_FET:AO3401A
- added Q2: AO3400A, Package_TO_SOT_SMD:SOT-23, symbol Transistor_FET:AO3400A
- added R5: 3900, Resistor_SMD:R_0805_2012Metric_Pad1.20x1.40mm_HandSolder, symbol Device:R
- added SW1: RotaryEncoder_Switch_MP, Rotary_Encoder:RotaryEncoder_Alps_EC12E-Switch_Vertical_H20mm_CircularMountingHoles, symbol Device:RotaryEncoder_Switch_MP
- added SW2: SW_NKK_GW12LJPCF, Button_Switch_THT:SW_NKK_GW12LJP, symbol Switch:SW_NKK_GW12LJPCF
- added U4, U5: TMP1075DGKR, DGK0008A_N, symbol TMP1075DGKR:TMP1075DGKR
- added Y1: Si570, Oscillator:Oscillator_SMD_SI570_SI571_HandSoldering, symbol Oscillator:Si570
- C1, C2: value 0.1uF -> C
- R1: value 330 -> R
- R2: value 100 -> R
- R3, R4: value 10k -> R
- U3: footprint DDPAK3_MC_MCH -> Package_TO_SOT_SMD:TO-263-2_TabPin1
Connections:
- net 5v_clock is gone; now on net GND: R1.2
- net 3.3v_AVDD: now also U1.64 (DIFFCLKENABLE), U1.70 (S/P_SELECT)
- net 3v_ldo: now also Y1.6 (Vcc); no longer R3.1
- net GND: now also C1.2, R3.2, TR2.4, TR2.5, C42.2, C43.2, C45.2, C46.2, C48.2, C50.2, C52.2, C53.2, R5.2, Y1.3 (GND); no longer C2.1
- net I_out_A: now also C1.1, C2.1, L2.1
- net I_out_B: now also R1.1
- net Q_out_A: now also C46.1, C47.1, L4.1
- net Q_out_B: now also R2.1
- net diffclockA: now also R3.1, Y1.4 (CLK+); no longer C1.2, R3.2, R4.1
- net diffclockB: now also R4.1, Y1.5 (CLK-); no longer C2.2
- net rf_outA: now also TR2.1
- net rf_outB: now also TR2.2
- net Lowpass_Q_out_A: now reaches TR2.3
- net Lowpass_Q_out_A: now also C51.2, C52.1, L6.2
- net Lowpass_I_out_A: now reaches TR2.6
- net Lowpass_I_out_A: now also C41.2, C45.1, L3.2
- net addrbus5: now reaches U1.14 (A5)
- net addrbus4: now reaches U1.15 (A4)
- net addrbus3: now reaches U1.16 (A3)
- net addrbus2: now reaches U1.17 (A2/IORESET)
- net addrbus1: now reaches U1.18 (A1/SDO)
- net addrbus0: now reaches U1.19 (A0/SDIO)
- net ioclock_AD9854: now reaches U1.20 (I/OUDCLK)
- net writeready_AD9854: now reaches U1.21 (WR*/SCLK)
- net readdata_AD9854: now reaches U1.22 (RD*/CS*)
- net at U1.55 (DACBP): now also C53.1
- net RESET_AD9854: now reaches U1.71 (MASTERRESET)
- new net: C2.2, C40.1, C42.1, L1.1, L2.2
- new net: C40.2, C41.1, C43.1, L1.2, L3.1
- new net: C47.2, C48.1, C49.1, L4.2, L5.1
- new net: C49.2, C50.1, C51.1, L5.2, L6.1
- new net dac_currentsetting: R5.1
- no-connect marks 6 -> 5
Other:
- added sheet Output_transformer_info (output_coupling_info.kicad_sch)
- added sheet refclock_info (refclock_info.kicad_sch)
- note added: "70 S/P SELECT Selects serial programming mode (logic low) or parallel programming mode (logic high). 56 DAC RSET Common Connection for Both I and Q DACs. Used to set the full-scale output current. RSET = 39.9/IOUT. Normal RSET range is from 8 kΩ (5 mA) to 2 kΩ (20 mA)"
- note added: "input & screen"
- note added: "relay"
- note added: "temp sensors"
- note removed: "OXCO clock - single 5vCMOS to differential"
- note removed: "TXCO clock - single 3.3vCMOS to differential"
- moved on the sheet: A1, TR2, U1, U2
